Commit message: update w irb1660 premoveit config

File: ROS_self_made_packages/robot_irb1660_id/urdf/robot_irb1660_id.urdf (robot description, URDF)
Before this commit: robot robot_irb1660_id, 8 links, 7 joints
Links:
- link base_link: geometry collision mesh filename=package://robot_irb1660_id/meshes/base_link.dae; visual mesh filename=package://robot_irb1660_id/meshes/base_link.dae
- link link_1: geometry collision mesh filename=package://robot_irb1660_id/meshes/link_1.dae; visual mesh filename=package://robot_irb1660_id/meshes/link_1.dae
- link link_2: geometry collision mesh filename=package://robot_irb1660_id/meshes/link_2.dae; visual mesh filename=package://robot_irb1660_id/meshes/link_2.dae
- link link_3: geometry collision mesh filename=package://robot_irb1660_id/meshes/link_3.dae; visual mesh filename=package://robot_irb1660_id/meshes/link_3.dae
- link link_4: geometry collision mesh filename=package://robot_irb1660_id/meshes/link_4.dae; visual mesh filename=package://robot_irb1660_id/meshes/link_4.dae
- link link_5: geometry collision mesh filename=package://robot_irb1660_id/meshes/link_5.dae; visual mesh filename=package://robot_irb1660_id/meshes/link_5.dae
- link link_6: geometry collision mesh filename=package://robot_irb1660_id/meshes/link_6.dae; visual mesh filename=package://robot_irb1660_id/meshes/link_6.dae
Joints:
- joint joint_3: origin xyz=0 0 0.475 rpy=0 0 0 -> xyz=0 0 0.700 rpy=0 0 0

Commit message: irb1660 urdf

File: ROS_self_made_packages/robot_irb1660_id/urdf/robot_irb1660_id.urdf (robot description, URDF)
Before this commit: robot robot_irb1660_id, 8 links, 7 joints
Links:
- link base_link: geometry collision mesh filename=package://robot_irb1660_id/meshes/base_link_bin.stl; visual mesh filename=package://robot_irb1660_id/meshes/base_link_bin.stl
- link link_1: geometry collision mesh filename=package://robot_irb1660_id/meshes/link_1_bin.stl; visual mesh filename=package://robot_irb1660_id/meshes/link_1_bin.stl
- link link_2: geometry collision mesh filename=package://robot_irb1660_id/meshes/link_2_bin.stl; visual mesh filename=package://robot_irb1660_id/meshes/link_2_bin.stl
- link link_3: geometry collision mesh filename=package://robot_irb1660_id/meshes/link_3_bin.stl; visual mesh filename=package://robot_irb1660_id/meshes/link_3_bin.stl
- link link_4: geometry collision mesh filename=package://robot_irb1660_id/meshes/link_4_bin.stl; visual mesh filename=package://robot_irb1660_id/meshes/link_4_bin.stl
- link link_5: geometry collision mesh filename=package://robot_irb1660_id/meshes/link_5_bin.stl; visual mesh filename=package://robot_irb1660_id/meshes/link_5_bin.stl
- link link_6: geometry collision mesh filename=package://robot_irb1660_id/meshes/link_6_bin.stl; visual mesh filename=package://robot_irb1660_id/meshes/link_6_bin.stl
Joints:
- joint joint_1: limit lower=-3.14159265359 upper=3.14159265359 effort=0 velocity=2.618 -> lower=-3.14159265359 upper=3.14159265359 effort=0 velocity=3.14159
- joint joint_2: limit lower=-1.0995 upper=1.9198 effort=0 velocity=2.7925 -> lower=-1.5708 upper=2.61799 effort=0 velocity=3.14159
- joint joint_3: limit lower=-4.1015 upper=0.9599 effort=0 velocity=2.9670 -> lower=-4.15388 upper=1.37881 effort=0 velocity=3.14159
- joint joint_4: limit lower=-3.4906 upper=3.4906 effort=0 velocity=5.5850 -> lower=-3.05433 upper=3.05433 effort=0 velocity=5.58505
- joint joint_5: limit lower=-2.0071 upper=2.0071 effort=0 velocity=6.9813 -> lower=-2.0944 upper=2.0944 effort=0 velocity=6.28319
- joint joint_6: limit lower=-6.9813 upper=6.9813 effort=0 velocity=7.854 -> lower=-6.98132 upper=6.98132 effort=0 velocity=8.72665

Commit message: irb1660 moveit configuratie

File: ROS_self_made_packages/robot_irb1660_id/urdf/robot_irb1660_id.urdf (robot description, URDF)
Before this commit: robot robot_irb1660_id, 8 links, 7 joints
Joints:
- joint joint_4: origin xyz=0.372 0 0 rpy=0 0 0 -> xyz=0.372 0 0.108 rpy=0 0 0

Commit message: irb1660 moveit configuratie

File: ROS_self_made_packages/robot_irb1660_id/urdf/robot_irb1660_id.urdf (robot description, URDF)
Before this commit: robot robot_irb1660_id, 8 links, 7 joints
Joints:
- joint joint_1: origin xyz=0 0 0 rpy=0 0 0 -> xyz=0 0 0.200 rpy=0 0 0

Commit message: irb1660 moveit configuratie

File: ROS_self_made_packages/robot_irb1660_id/urdf/robot_irb1660_id.urdf (robot description, URDF)
Before this commit: robot robot_irb1660_id, 8 links, 7 joints
Joints:
- joint joint_1: origin xyz=0 0 0.200 rpy=0 0 0 -> xyz=0 0 0.134 rpy=0 0 0
- joint joint_2: origin xyz=0.15 0 0.4865 rpy=0 0 0 -> xyz=0.15 0 0.3525 rpy=0 0 0

Commit message: irb1660 moveit configuratie

File: ROS_self_made_packages/robot_irb1660_id/urdf/robot_irb1660_id.urdf (robot description, URDF)
Before this commit: robot robot_irb1660_id, 8 links, 7 joints
Joints:
- joint joint_2: origin xyz=0.15 0 0.3525 rpy=0 0 0 -> xyz=0.15 -0.221 0.3525 rpy=0 0 0
- joint joint_3: origin xyz=0 0 0.700 rpy=0 0 0 -> xyz=0 0.0065 0.700 rpy=0 0 0
- joint joint_4: origin xyz=0.372 0 0.108 rpy=0 0 0 -> xyz=0.128 0.2145 0.108 rpy=0 0 0
- joint joint_5: origin xyz=0.306 0 0 rpy=0 0 0 -> xyz=0.550 0 0 rpy=0 0 0
- joint joint_6: origin xyz=0.135 0 0 rpy=0 0 0 -> xyz=0.135 0 0 rpy=0.0 0 0
