Commit message: update irb1660id for fieldlab

File: ROS_self_made_packages/robot_irb1660_id/urdf/robot_irb1660_id_fieldlab.urdf (robot description, URDF)
Before this commit: robot robot_irb1660_id, 8 links, 7 joints
Links:
- link link_1: geometry collision mesh filename=package://robot_irb1660_id/meshes/link_1_bin_zeroed.stl; visual mesh filename=package://robot_irb1660_id/meshes/link_1_bin_zeroed.stl
- link link_2: geometry collision mesh filename=package://robot_irb1660_id/meshes/link_2_bin_zeroed.stl; visual mesh filename=package://robot_irb1660_id/meshes/link_2_bin_zeroed.stl
- link link_3: geometry collision mesh filename=package://robot_irb1660_id/meshes/link_3_bin_zeroed.stl; visual mesh filename=package://robot_irb1660_id/meshes/link_3_bin_zeroed.stl
- link link_4: geometry collision mesh filename=package://robot_irb1660_id/meshes/link_4_bin_zeroed.stl; visual mesh filename=package://robot_irb1660_id/meshes/link_4_bin_zeroed.stl
- link link_5: geometry collision mesh filename=package://robot_irb1660_id/meshes/link_5_bin_zeroed.stl; visual mesh filename=package://robot_irb1660_id/meshes/link_5_bin_zeroed.stl
- link link_6: geometry collision mesh filename=package://robot_irb1660_id/meshes/link_6_bin_zeroed.stl; visual mesh filename=package://robot_irb1660_id/meshes/link_6_bin_zeroed.stl
Joints:
- joint joint_1: limit lower=-3.14159265359 upper=3.14159265359 effort=0 velocity=3.14159 -> lower=-3.14159 upper=3.14159 effort=0 velocity=2.47837; origin xyz=0 0 0.134 rpy=0 0 0 -> xyz=0 0 0.124 rpy=0 0 0
- joint joint_2: limit lower=-1.5708 upper=2.61799 effort=0 velocity=3.14159 -> lower=-1.5708 upper=2.61799 effort=0 velocity=2.46091; origin xyz=0.15 -0.221 0.3525 rpy=0 0 0 -> xyz=0.15 -0.107 0.3625 rpy=0 0 0
- joint joint_3: limit lower=-4.15388 upper=1.37881 effort=0 velocity=3.14159 -> lower=-4.15388 upper=1.37881 effort=0 velocity=2.74017; origin xyz=0 0.0065 0.700 rpy=0 0 0 -> xyz=0 0 0.7 rpy=0 0 0
- joint joint_4: origin xyz=0 0.2145 0.108 rpy=0 0 0 -> xyz=0.128 0.107 0.108 rpy=0 0 0
- joint joint_5: limit lower=-2.0944 upper=2.0944 effort=0 velocity=6.28319 -> lower=-2.0944 upper=2.0944 effort=0 velocity=5.74213; origin xyz=0.678 0 0 rpy=0 0 0 -> xyz=0.55 0 0 rpy=0 0 0
- joint joint_6: limit lower=-6.98132 upper=6.98132 effort=0 velocity=8.72665 -> lower=-6.98132 upper=6.98132 effort=0 velocity=6.47517
- joint joint_6-tool0: origin xyz=0 0 0 rpy=0 1.57079632679 0 -> xyz=0 0 0 rpy=0 0 0

File: ROS_self_made_packages/robot_irb1660_id/urdf/robot_irb1660_id_zeroed.urdf (robot description, URDF)
Before this commit: robot robot_irb1660_id, 8 links, 7 joints
Links:
- link link_1: geometry collision mesh filename=package://robot_irb1660_id/meshes/link_1_bin_zeroed.stl; visual mesh filename=package://robot_irb1660_id/meshes/link_1_bin_zeroed.stl
- link link_2: geometry collision mesh filename=package://robot_irb1660_id/meshes/link_2_bin_zeroed.stl; visual mesh filename=package://robot_irb1660_id/meshes/link_2_bin_zeroed.stl
- link link_3: geometry collision mesh filename=package://robot_irb1660_id/meshes/link_3_bin_zeroed.stl; visual mesh filename=package://robot_irb1660_id/meshes/link_3_bin_zeroed.stl
- link link_4: geometry collision mesh filename=package://robot_irb1660_id/meshes/link_4_bin_zeroed.stl; visual mesh filename=package://robot_irb1660_id/meshes/link_4_bin_zeroed.stl
- link link_5: geometry collision mesh filename=package://robot_irb1660_id/meshes/link_5_bin_zeroed.stl; visual mesh filename=package://robot_irb1660_id/meshes/link_5_bin_zeroed.stl
- link link_6: geometry collision mesh filename=package://robot_irb1660_id/meshes/link_6_bin_zeroed.stl; visual mesh filename=package://robot_irb1660_id/meshes/link_6_bin_zeroed.stl
Joints:
- joint joint_1: limit lower=-3.14159265359 upper=3.14159265359 effort=0 velocity=3.14159 -> lower=-3.14159 upper=3.14159 effort=0 velocity=2.47837; origin xyz=0 0 0.134 rpy=0 0 0 -> xyz=0 0 0.124 rpy=0 0 0
- joint joint_2: limit lower=-1.5708 upper=2.61799 effort=0 velocity=3.14159 -> lower=-1.5708 upper=2.61799 effort=0 velocity=2.46091; origin xyz=0.15 -0.221 0.3525 rpy=0 0 0 -> xyz=0.15 -0.107 0.3625 rpy=0 0 0
- joint joint_3: limit lower=-4.15388 upper=1.37881 effort=0 velocity=3.14159 -> lower=-4.15388 upper=1.37881 effort=0 velocity=2.74017; origin xyz=0 0.0065 0.700 rpy=0 0 0 -> xyz=0 0 0.7 rpy=0 0 0
- joint joint_4: origin xyz=0 0.2145 0.108 rpy=0 0 0 -> xyz=0.128 0.107 0.108 rpy=0 0 0
- joint joint_5: limit lower=-2.0944 upper=2.0944 effort=0 velocity=6.28319 -> lower=-2.0944 upper=2.0944 effort=0 velocity=5.74213; origin xyz=0.678 0 0 rpy=0 0 0 -> xyz=0.55 0 0 rpy=0 0 0
- joint joint_6: limit lower=-6.98132 upper=6.98132 effort=0 velocity=8.72665 -> lower=-6.98132 upper=6.98132 effort=0 velocity=6.47517
- joint joint_6-tool0: origin xyz=0 0 0 rpy=0 1.57079632679 0 -> xyz=0 0 0 rpy=1 0 0

Commit message: abb robot calibration package start

File: ROS_self_made_packages/robot_irb1660_id/urdf/robot_irb1660_id_fieldlab.urdf (robot description, URDF)
Before this commit: robot robot_irb1660_id, 8 links, 7 joints
Joints:
- joint joint_1: limit lower=-3.14159 upper=3.14159 effort=0 velocity=2.47837 -> lower=-3.14159 upper=3.14159 effort=0 velocity=3.14159
- joint joint_2: limit lower=-1.5708 upper=2.61799 effort=0 velocity=2.46091 -> lower=-1.5708 upper=2.61799 effort=0 velocity=3.14159
- joint joint_3: limit lower=-4.15388 upper=1.37881 effort=0 velocity=2.74017 -> lower=-4.15388 upper=1.37881 effort=0 velocity=3.14159
- joint joint_5: limit lower=-2.0944 upper=2.0944 effort=0 velocity=5.74213 -> lower=-2.0944 upper=2.0944 effort=0 velocity=6.28319
- joint joint_6: limit lower=-6.98132 upper=6.98132 effort=0 velocity=6.47517 -> lower=-6.98132 upper=6.98132 effort=0 velocity=8.72665
