Commit message: abb robot calibration package

File: ROS_self_made_packages/robot_irb1660_id/urdf/robot_irb1660_id_fieldlab_camera.urdf (robot description, URDF)
Before this commit: robot robot_irb1660_id, 8 links, 7 joints
Links:
- added link camera_link; collision box size=0.2 0.2 0.2; visual box size=0.2 0.2 0.2
Joints:
- added joint camera-baselink: type fixed, parent base_link, child camera_link, origin xyz=2.0 0 0 rpy=0 0 0

Commit message: abb robot calibration package

File: ROS_self_made_packages/robot_irb1660_id/urdf/robot_irb1660_id_fieldlab_camera.urdf (robot description, URDF)
Before this commit: robot robot_irb1660_id, 9 links, 8 joints
Links:
- link camera_link: mass None -> 1; geometry 
Joints:
- joint camera-baselink: origin xyz=2.0 0 0 rpy=0 0 0 -> xyz=0 0 0 rpy=0 0 0

Commit message: update urdf for camera frame definitions

File: ROS_self_made_packages/robot_irb1660_id/urdf/robot_irb1660_id_fieldlab_camera.urdf (robot description, URDF)
Before this commit: robot robot_irb1660_id, 9 links, 8 joints
Links:
- added link camera_optical_frame
- link camera_link: mass 1 -> None; geometry visual box size=0.2 0.2 0.2
Joints:
- removed joint camera-baselink
- added joint camera_joint: type fixed, parent base_link, child camera_link, origin xyz=2.0 0 1.0 rpy=0 -3.14159 0
- added joint camera_optical_joint: type fixed, parent camera_link, child camera_optical_frame, origin xyz=0 0 0 rpy=0 0 0

Commit message: Update After test on actual robot

File: ROS_self_made_packages/robot_irb1660_id/urdf/robot_irb1660_id_fieldlab_camera.urdf (robot description, URDF)
Before this commit: robot robot_irb1660_id, 10 links, 9 joints
Joints:
- joint camera_joint: origin xyz=2.0 0 1.0 rpy=0 -3.14159 0 -> xyz=3.5 -1.10 -0.35 rpy=0 -3.14159 0
