Commit message: urdf w tool

File: abb_ros/src/abb_irb1660_support/urdf/irb1660_external_camera.urdf (robot description, URDF)
Before this commit: robot irb1660_6_155, 10 links, 9 joints
Links:
- link tool0: geometry collision mesh filename=package://abb_irb1660_support/meshes/tools/tool_sks_FP8i-L.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; visual mesh filename=package://abb_irb1660_support/meshes/tools/tool_sks_FP8i-L.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

Commit message: industrial_core offset support

File: abb_ros/src/abb_irb1660_support/urdf/irb1660_external_camera.urdf (robot description, URDF)
Before this commit: robot irb1660_6_155, 10 links, 9 joints
Joints:
- joint camera_joint: origin xyz=2.85 1.43 0.12 rpy=0 -3.14159 0 -> xyz=2.85 0 0.5 rpy=0 -3.14159 0

Commit message: load_calibration_offsets.py

File: abb_ros/src/abb_irb1660_support/urdf/irb1660_external_camera.urdf (robot description, URDF)
Before this commit: robot irb1660_6_155, 10 links, 9 joints
Links:
- added link external_axis_object; collision box size=0.45 1.60 1.05; visual box size=0.45 1.60 1.05
- added link front_of_cel_link
- added link ground_object; collision box size=4 0.05 3.25; visual box size=4 0.05 3.25
- added link wall_back_object; collision box size=3.25 0.05 2.5; visual box size=3.25 0.05 2.5
- added link wall_left_object; collision box size=4 0.05 2.5; visual box size=4 0.05 2.5
- added link wall_right_object; collision box size=4 0.05 2.5; visual box size=4 0.05 2.5
Joints:
- added joint external_axis_joint: type fixed, parent front_of_cel_link, child external_axis_object, origin xyz=-0.75 0 0 rpy=0 0 0
- added joint front_of_cel_joint: type fixed, parent base_link, child front_of_cel_link, origin xyz=2 0 -0.655 rpy=0 0 0
- added joint front_to_back_wall_joint: type fixed, parent front_of_cel_link, child wall_back_object, origin xyz=-4 0 0 rpy=0 0 0
- added joint front_to_left_wall_joint: type fixed, parent front_of_cel_link, child wall_left_object, origin xyz=0 -1.625 0 rpy=0 0 0
- added joint front_to_right_wall_joint: type fixed, parent front_of_cel_link, child wall_right_object, origin xyz=0 1.625 0 rpy=0 0 0
- added joint ground_joint: type fixed, parent front_of_cel_link, child ground_object, origin xyz=-2 0 0 rpy=0 0 0
