Commit message: multiple cameras configuration and poses

File: abb_ros/src/abb_irb1660_support/urdf/irb1660_6_155_multiple_camera.urdf (robot description, URDF)
Before this commit: robot irb1660_6_155, 19 links, 18 joints
Joints:
- joint external_axis_joint: origin xyz=-0.75 0 0 rpy=0 0 0 -> xyz=0.993 0 0 rpy=0 0 0; parent front_of_cel_link -> base_link
- joint external_camera_joint: origin xyz=3.02 0 0.79 rpy=0 -3.14159 0 -> xyz=2.439 0.60 0.354 rpy=0 0 4.75
- joint external_camera_optical_joint: origin xyz=0.025 0 0 rpy=0 0 0 -> xyz=0.010 0 0.010 rpy=0 0 0
- joint led_joint: origin xyz=0.463 0.0 -0.120 rpy=0 0 0 -> xyz=0.463 0.0 -0.110 rpy=0 0 0
- joint mounted_camera_joint: origin xyz=0.115 0 0.112 rpy=0 0 0 -> xyz=0.095 0 0.075 rpy=0 0 0
- joint mounted_camera_optical_joint: origin xyz=0.025 0 0 rpy=0 0 0 -> xyz=0.010 0 0.010 rpy=0 0 0
