Commit message: intital calibration results

File: abb_ros/src/fieldlab_cel3_calib/config/calibrated_urdfs/calibrated_test2.urdf (robot description, URDF)
Before this commit: robot irb1660_6_155, 17 links, 16 joints
Joints:
- joint camera_joint: origin xyz=0.115 0 0.112 rpy=0 0 0 -> xyz=3.02 0.50 0.50 rpy=0 0 -2.7488909; parent link_5 -> base_link
