Commit message: calibration params

File: fieldlab_cel3_calib/calibration_multiple_cams/calibrated_fieldlab_cel3_calibration_output.urdf (robot description, URDF)
Before this commit: robot irb1660_6_155, 19 links, 18 joints
Joints:
- joint external_camera_optical_joint: origin xyz=0.010 0 0.010 rpy=0 0 0 -> xyz=0.01000000 0.00000000 0.01000000 rpy=0.00000000 0.00000000 0.00000000
- joint mounted_camera_optical_joint: origin xyz=0.010 0 0.010 rpy=0 0 0 -> xyz=0.01000000 0.00000000 0.01000000 rpy=0.00000000 0.00000000 0.00000000
